Commit message: 車両は走るようになった。RVizでFixedFieldを正しく設定して表示を確認。point lioがlidarからのデータにtimestampが含まれていないためエラー。修正としてadd_time_field.pyを追加

File: src/sim/sim_gazebo/urdf/four_wheel_car.urdf (robot description, URDF)
Before this commit: robot four_wheel_car, 7 links, 6 joints
Links:
- added link imu_link, mass 0.01
- added link lidar_link, mass 0.1; collision cylinder length=0.07 radius=0.05; visual cylinder length=0.07 radius=0.05
Joints:
- added joint imu_joint: type fixed, parent lidar_link, child imu_link, origin xyz=0 0 0 rpy=0 0 0
- added joint lidar_joint: type fixed, parent base_link, child lidar_link, origin xyz=0.2 0.0 0.25 rpy=0 0 0
